File: sensors.kicad_sch (KiCad schematic)
At the start: 21 parts, among them J1 Conn_01x07, U1 TCRT5000, U2 TCRT5000, U3 TCRT5000, U4 TCRT5000, U5 TCRT5000

Commit message: Add files via upload
Parts:
- C1, C2, C3, C4, C5: value C -> 0.1 µF
- R1, R3, R5, R7, R9: value R -> 470
- R10, R2, R4, R6, R8: value R -> 220
Changed lines of the file:
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@@
       (effects (font (size 1.27 1.27)) (justify left))
     )
-    (property "Value" "C" (at 146.05 91.44 0)
+    (property "Value" "0.1 µF" (at 146.05 91.44 0)
       (effects (font (size 1.27 1.27)) (justify left))
     )
@@
       (effects (font (size 1.27 1.27)))
     )
-    (property "Value" "R" (at 83.82 140.97 90)
+    (property "Value" "220" (at 83.82 140.97 90)
       (effects (font (size 1.27 1.27)))
     )
@@
       (effects (font (size 1.27 1.27)) (justify left))
     )
-    (property "Value" "R" (at 41.91 139.7 0)
+    (property "Value" "470" (at 41.91 139.7 0)
       (effects (font (size 1.27 1.27)) (justify left))
     )
@@
       (effects (font (size 1.27 1.27)) (justify left))
     )
-    (property "Value" "C" (at 74.93 44.45 0)
+    (property "Value" "0.1 µF" (at 74.93 44.45 0)
       (effects (font (size 1.27 1.27)) (justify left))
     )
@@
       (effects (font (size 1.27 1.27)))
     )
-    (property "Value" "R" (at 153.67 93.98 90)
+    (property "Value" "220" (at 153.67 93.98 90)
       (effects (font (size 1.27 1.27)))
     )
@@
       (effects (font (size 1.27 1.27)) (justify left))
     )
-    (property "Value" "R" (at 41.91 92.71 0)
+    (property "Value" "470" (at 41.91 92.71 0)
       (effects (font (size 1.27 1.27)) (justify left))
     )
@@
       (effects (font (size 1.27 1.27)))
     )
-    (property "Value" "R" (at 82.55 46.99 90)
+    (property "Value" "220" (at 82.55 46.99 90)
       (effects (font (size 1.27 1.27)))
     )
@@
       (effects (font (size 1.27 1.27)) (justify left))
     )
-    (property "Value" "C" (at 146.05 43.18 0)
+    (property "Value" "0.1 µF" (at 146.05 43.18 0)
       (effects (font (size 1.27 1.27)) (justify left))
     )
@@
       (effects (font (size 1.27 1.27)))
     )
-    (property "Value" "R" (at 83.82 93.98 90)
+    (property "Value" "220" (at 83.82 93.98 90)
       (effects (font (size 1.27 1.27)))
     )
@@
       (effects (font (size 1.27 1.27)) (justify left))
     )
-    (property "Value" "C" (at 76.2 138.43 0)
+    (property "Value" "0.1 µF" (at 76.2 138.43 0)
       (effects (font (size 1.27 1.27)) (justify left))
     )
@@
       (effects (font (size 1.27 1.27)))
     )
-    (property "Value" "R" (at 153.67 45.72 90)
+    (property "Value" "220" (at 153.67 45.72 90)
       (effects (font (size 1.27 1.27)))
     )
@@
       (effects (font (size 1.27 1.27)) (justify left))
     )
-    (property "Value" "R" (at 111.76 44.45 0)
+    (property "Value" "470" (at 111.76 44.45 0)
       (effects (font (size 1.27 1.27)) (justify left))
     )
@@
       (effects (font (size 1.27 1.27)) (justify left))
     )
-    (property "Value" "R" (at 40.64 45.72 0)
+    (property "Value" "470" (at 40.64 45.72 0)
       (effects (font (size 1.27 1.27)) (justify left))
     )
@@
       (effects (font (size 1.27 1.27)) (justify left))
     )
-    (property "Value" "R" (at 111.76 92.71 0)
+    (property "Value" "470" (at 111.76 92.71 0)
       (effects (font (size 1.27 1.27)) (justify left))
     )
@@
       (effects (font (size 1.27 1.27)) (justify left))
     )
-    (property "Value" "C" (at 76.2 91.44 0)
-      (effects (font (size 1.27 1.27)) (justify left))
-    )
+    (property "Value" "0.1 µF" (at 76.2 91.44 0)
+      (effects (font (size 1.27 1.27)) (justify left))
+    )
