File: TCRT5000 seperated.kicad_pcb (KiCad board)
At the start: 2 copper layers, 57.7 x 30.6 mm, 14 parts, among them J1 Conn_01x03, J2 Conn_01x03, U1 TCRT5000, U2 TCRT5000

Commit message: Add files via upload
Parts:
- moved R3 0.73 mm to (105.9, 92.6)
- moved C1 0.45 mm to (110.4, 92.5)
Routing:
- net +3.3V: track 62.0 -> 58.9 mm
- net GND: track 13.8 -> 12.2 mm
- net Sensor 02R: track 5.18 -> 5.69 mm

Commit message: Add files via upload
Parts:
- moved J2 25.6 mm to (125.7, 89.0)
- moved C2 25.6 mm to (129.9, 92.3)
- moved H2 25.6 mm to (128.5, 82.9)
- moved R4 25.6 mm to (124.0, 102.1)
- moved R5 25.6 mm to (124.0, 97.1)
- moved R6 25.6 mm to (125.4, 92.3)
- moved U2 25.6 mm to (129.0, 99.5)
- moved H1 5.79 mm to (114.6, 83.1)
- moved C1 5.33 mm to (115.8, 92.5)
- moved J1 5.33 mm to (111.3, 89.4)
- moved R1 5.33 mm to (109.9, 102.2)
- moved R2 5.33 mm to (109.9, 97.1)
- moved U1 5.33 mm to (114.6, 99.3)
- moved R3 5.33 mm to (111.2, 92.6)
Routing:
- net (no net): vias 0 -> 19
Other:
- board size 57.7 x 30.6 mm -> 27.2 x 30.5 mm
