File: PCB/SensorBoardBackup/TCRT5000 seperated.kicad_sch (KiCad schematic)
At the start: 14 parts, among them J1 Conn_01x03, J2 Conn_01x03, U1 TCRT5000, U2 TCRT5000

Commit message: Version that was resubmitted
Parts:
- removed C2: C, Capacitor_SMD:C_1206_3216Metric, symbol Device:C
- removed H2: MountingHole, MountingHole:MountingHole_3mm, symbol Mechanical:MountingHole
- removed J2: Conn_01x03, Connector_PinHeader_2.54mm:PinHeader_1x03_P2.54mm_Vertical, symbol Connector_Generic:Conn_01x03
- removed R4: 90, Resistor_SMD:R_0805_2012Metric, symbol Device:R
- removed R5: 3.9k, Resistor_SMD:R_0805_2012Metric, symbol Device:R
- removed R6: R, Resistor_SMD:R_0805_2012Metric, symbol Device:R
- removed U2: TCRT5000, Footprints:OPTO_TCRT5000, symbol TCRT5000:TCRT5000
